Commit message: fixing pinnochio import for ik unit tests

File: source/isaaclab/test/controllers/urdfs/test_urdf_two_link_robot.urdf (robot description, URDF)
Before this commit: robot test_two_link_robot, 4 links, 3 joints
Links:
- link base_link: mass 1.0 -> None; geometry 
- link link_1: mass 1.0 -> None; geometry 
- link link_2: mass 1.0 -> None; geometry 
- link world: mass 0.001 -> None
